Commit message: Fixed CMakeList for including custom controller

File: franka_robot.urdf (robot description, URDF)
Before this commit: robot fr3, 26 links, 25 joints
Links:
- removed link fr3_link0_accelerometer_bottom
- removed link fr3_link0_accelerometer_top
- removed link fr3_link1_accelerometer_bottom
- removed link fr3_link1_accelerometer_top
- removed link fr3_link2_accelerometer_bottom
- removed link fr3_link2_accelerometer_top
- removed link fr3_link3_accelerometer_bottom
- removed link fr3_link3_accelerometer_top
- removed link fr3_link4_accelerometer_bottom
- removed link fr3_link4_accelerometer_top
- removed link fr3_link5_accelerometer_bottom
- removed link fr3_link5_accelerometer_top
- link fr3_hand: mass 0.6544 -> 0.73
- link fr3_leftfinger: mass 0.0291 -> 0.015
- link fr3_link0: geometry collision mesh filename=package://franka_description/meshes/robot_arms/fr3/collisio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; visual mesh filename=package://franka_description/meshes/robot_arms/fr3/visual/l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
- link fr3_link1: geometry collision mesh filename=package://franka_description/meshes/robot_arms/fr3/collisio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; visual mesh filename=package://franka_description/meshes/robot_arms/fr3/visual/l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
- link fr3_link2: geometry collision mesh filename=package://franka_description/meshes/robot_arms/fr3/collisio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; visual mesh filename=package://franka_description/meshes/robot_arms/fr3/visual/l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
- link fr3_link3: geometry collision mesh filename=package://franka_description/meshes/robot_arms/fr3/collisio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; visual mesh filename=package://franka_description/meshes/robot_arms/fr3/visual/l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
- link fr3_link4: geometry collision mesh filename=package://franka_description/meshes/robot_arms/fr3/collisio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; visual mesh filename=package://franka_description/meshes/robot_arms/fr3/visual/l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
- link fr3_link5: geometry collision mesh filename=package://franka_description/meshes/robot_arms/fr3/collisio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; visual mesh filename=package://franka_description/meshes/robot_arms/fr3/visual/l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
- link fr3_link6: geometry collision mesh filename=package://franka_description/meshes/robot_arms/fr3/collisio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; visual mesh filename=package://franka_description/meshes/robot_arms/fr3/visual/l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
- link fr3_link7: geometry collision mesh filename=package://franka_description/meshes/robot_arms/fr3/collisio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; visual mesh filename=package://franka_description/meshes/robot_arms/fr3/visual/l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
- link fr3_rightfinger: mass 0.0291 -> 0.015
Joints:
- removed joint fr3_link0_accelerometer_bottom_joint
- removed joint fr3_link0_accelerometer_top_joint
- removed joint fr3_link1_accelerometer_bottom_joint
- removed joint fr3_link1_accelerometer_top_joint
- removed joint fr3_link2_accelerometer_bottom_joint
- removed joint fr3_link2_accelerometer_top_joint
- removed joint fr3_link3_accelerometer_bottom_joint
- removed joint fr3_link3_accelerometer_top_joint
- removed joint fr3_link4_accelerometer_bottom_joint
- removed joint fr3_link4_accelerometer_top_joint
- removed joint fr3_link5_accelerometer_bottom_joint
- removed joint fr3_link5_accelerometer_top_joint
- joint fr3_finger_joint2: axis 0 1 0 -> 0 -1 0; origin xyz=0 0 0.0584 rpy=0 0 3.141592653589793 -> xyz=0 0 0.0584 rpy=0 0 0
- joint fr3_joint1: limit lower=-2.9007 upper=2.9007 effort=87.0 velocity=2.62 -> lower=-2.7437 upper=2.7437 effort=87.0 velocity=2.62
- joint fr3_joint2: limit lower=-1.8361 upper=1.8361 effort=87.0 velocity=2.62 -> lower=-1.7837 upper=1.7837 effort=87.0 velocity=2.62
- joint fr3_joint4: limit lower=-3.077 upper=-0.1169 effort=87.0 velocity=2.62 -> lower=-3.0421 upper=-0.1518 effort=87.0 velocity=2.62
- joint fr3_joint5: limit lower=-2.8763 upper=2.8763 effort=12.0 velocity=5.26 -> lower=-2.8065 upper=2.8065 effort=12.0 velocity=5.26
- joint fr3_joint6: limit lower=0.4398 upper=4.6216 effort=12.0 velocity=4.18 -> lower=0.5445 upper=4.5169 effort=12.0 velocity=4.18
- joint fr3_joint7: limit lower=-3.0508 upper=3.0508 effort=12.0 velocity=5.26 -> lower=-3.0159 upper=3.0159 effort=12.0 velocity=5.26
